File: LTC4162/LTC4162.kicad_sch (KiCad schematic)
At the start: 17 parts, among them J1 Conn_01x02, J2 Conn_01x02, J3 Conn_01x02, Q6 FDMC8327L, Q7 2N7002

Commit message: Add files via upload
Other:
- note added: "- CLP / CLN (Chân 5, 4): V = ~9V (Đo dòng vào) | I = ~µA (Sụt áp tối đa giữa 2 chân là 32mV) - CSP / CSN (Chân 21, 20): V = 2.5V - 4.2V (Đo dòng sạc pin) | I = ~µA (Sụt áp tối đa giữa 2 chân là 32mV) - BATSENS+ (Chân 19): V = 2.5V - 4.2V (Đo áp pin) | I = 54µA - 100µA"
- note added: "- INFET / BATFET (Chân 6, 22): V ≈ 15V - 20V (Áp kích Charge Pump) | I = ~µA - INTVCC (Chân 2): V = 5V | I = (LDO) - VCC2P5 (Chân 8): V = 2.5V | I = (LDO)"
- note added: "- VIN (Chân 7): V = 9V (Max 35V) | I = 2.5A (Dòng vào từ Solar) - VOUT (Chân 27, 28): V = 9V (Max 35V) | I = 2.5A - SW (Chân 25, 26): V = 0V ↔ 9V (Dao động 1.5MHz) | I = 3.2A - PGND (Chân 23, 24): V = 0V | I = 3.2A"
- note added: "1. NHÓM CHÂN CÔNG SUẤT (DÒNG LỚN)"
- note added: "2. NHÓM CHÂN ĐO LƯỜNG (DÒNG NHỎ)"
- note added: "3. NHÓM CHÂN ĐIỀU KHIỂN (ÁP CAO, DÒNG NHỎ)"
- moved on the sheet: B4, C14, C15, C16, C17, C5, J1, J2, J3, L2, NTCS0402E3103FLT2, Q6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

Commit message: Add files via upload
Parts:
- B4: footprint QFN50P400X500X80-29N-D -> LTC4162:QFN50P400X500X80-29N-D
Changed lines of the file:
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@@
+				)
+			)
+			(project "TTT"
+				(path "/990e0fce-b73a-47af-aaa3-74ef9b552d39/22221f63-b32d-4372-b662-a2ce74004c9b"
+					(reference "#PWR08")
+					(unit 1)
 				)
 			)
@@
 				)
 			)
+			(project "TTT"
+				(path "/990e0fce-b73a-47af-aaa3-74ef9b552d39/22221f63-b32d-4372-b662-a2ce74004c9b"
+					(reference "C3")
+					(unit 1)
+				)
+			)
 		)
 	)
@@
 				(path "/3c29357a-68d2-4983-bb91-6d3951934863"
 					(reference "NTCS0402E3103FLT2")
+					(unit 1)
+				)
+			)
+			(project "TTT"
+				(path "/990e0fce-b73a-47af-aaa3-74ef9b552d39/22221f63-b32d-4372-b662-a2ce74004c9b"
+					(reference "NTCS0402E3103FLT1")
 					(unit 1)
 				)
@@
 				)
 			)
+			(project "TTT"
+				(path "/990e0fce-b73a-47af-aaa3-74ef9b552d39/22221f63-b32d-4372-b662-a2ce74004c9b"
+					(reference "Q2")
+					(unit 1)
+				)
+			)
 		)
 	)
@@
 				)
 			)
+			(project "TTT"
+				(path "/990e0fce-b73a-47af-aaa3-74ef9b552d39/22221f63-b32d-4372-b662-a2ce74004c9b"
+					(reference "#PWR05")
+					(unit 1)
+				)
+			)
 		)
 	)
@@
 			)
 		)
-		(property "Footprint" "QFN50P400X500X80-29N-D"
+		(property "Footprint" "LTC4162:QFN50P400X500X80-29N-D"
 			(at 187.96 97.79 0)
 			(hide yes)
@@
 				(path "/3c29357a-68d2-4983-bb91-6d3951934863"
 					(reference "B4")
+					(unit 1)
+				)
+			)
+			(project "TTT"
+				(path "/990e0fce-b73a-47af-aaa3-74ef9b552d39/22221f63-b32d-4372-b662-a2ce74004c9b"
+					(reference "B2")
 					(unit 1)
 				)
@@
 				)
 			)
+			(project "TTT"
+				(path "/990e0fce-b73a-47af-aaa3-74ef9b552d39/22221f63-b32d-4372-b662-a2ce74004c9b"
+					(reference "J3")
+					(unit 1)
+				)
+			)
 		)
 	)
@@
 				(path "/3c29357a-68d2-4983-bb91-6d3951934863"
 					(reference "L2")
+					(unit 1)
+				)
+			)
+			(project "TTT"
+				(path "/990e0fce-b73a-47af-aaa3-74ef9b552d39/22221f63-b32d-4372-b662-a2ce74004c9b"
+					(reference "L1")
 					(unit 1)
 				)
@@
 				)
 			)
+			(project "TTT"
+				(path "/990e0fce-b73a-47af-aaa3-74ef9b552d39/22221f63-b32d-4372-b662-a2ce74004c9b"
+					(reference "#PWR01")
+					(unit 1)
+				)
+			)
 		)
 	)
@@
 				)
 			)
+			(project "TTT"
+				(path "/990e0fce-b73a-47af-aaa3-74ef9b552d39/22221f63-b32d-4372-b662-a2ce74004c9b"
+					(reference "#PWR016")
+					(unit 1)
+				)
+			)
 		)
 	)
@@
 				)
 			)
+			(project "TTT"
+				(path "/990e0fce-b73a-47af-aaa3-74ef9b552d39/22221f63-b32d-4372-b662-a2ce74004c9b"
+					(reference "J2")
+					(unit 1)
+				)
+			)
 		)
 	)
@@
 				)
 			)
+			(project "TTT"
+				(path "/990e0fce-b73a-47af-aaa3-74ef9b552d39/22221f63-b32d-4372-b662-a2ce74004c9b"
+					(reference "#PWR03")
+					(unit 1)
+				)
+			)
 		)
 	)
@@
 				)
 			)
+			(project "TTT"
+				(path "/990e0fce-b73a-47af-aaa3-74ef9b552d39/22221f63-b32d-4372-b662-a2ce74004c9b"
+					(reference "C7")
+					(unit 1)
+				)
+			)
 		)
 	)
@@
 				)
 			)
+			(project "TTT"
+				(path "/990e0fce-b73a-47af-aaa3-74ef9b552d39/22221f63-b32d-4372-b662-a2ce74004c9b"
+					(reference "#PWR02")
+					(unit 1)
+				)
+			)
 		)
 	)
@@
 				(path "/3c29357a-68d2-4983-bb91-6d3951934863"
 					(reference "Q7")
+					(unit 1)
+				)
+			)
+			(project "TTT"
+				(path "/990e0fce-b73a-47af-aaa3-74ef9b552d39/22221f63-b32d-4372-b662-a2ce74004c9b"
+					(reference "Q3")
 					(unit 1)
 				)
@@
 				)
 			)
+			(project "TTT"
+				(path "/990e0fce-b73a-47af-aaa3-74ef9b552d39/22221f63-b32d-4372-b662-a2ce74004c9b"
+					(reference "R2")
+					(unit 1)
+				)
+			)
 		)
 	)
@@
 				)
 			)
+			(project "TTT"
+				(path "/990e0fce-b73a-47af-aaa3-74ef9b552d39/22221f63-b32d-4372-b662-a2ce74004c9b"
+					(reference "Rsnsi1")
+					(unit 1)
+				)
+			)
 		)
 	)
@@
 				)
 			)
+			(project "TTT"
+				(path "/990e0fce-b73a-47af-aaa3-74ef9b552d39/22221f63-b32d-4372-b662-a2ce74004c9b"
+					(reference "C4")
+					(unit 1)
+				)
+			)
 		)
 	)
@@
 				)
 			)
+			(project "TTT"
+				(path "/990e0fce-b73a-47af-aaa3-74ef9b552d39/22221f63-b32d-4372-b662-a2ce74004c9b"
+					(reference "C6")
+					(unit 1)
+				)
+			)
 		)
 	)
@@
 			(project "LTC4162"
 				(path "/3c29357a-68d2-4983-bb91-6d3951934863"
+					(reference "C5")
+					(unit 1)
+				)
+			)
+			(project "TTT"
+				(path "/990e0fce-b73a-47af-aaa3-74ef9b552d39/22221f63-b32d-4372-b662-a2ce74004c9b"
 					(reference "C5")
 					(unit 1)
@@
 				)
 			)
+			(project "TTT"
+				(path "/990e0fce-b73a-47af-aaa3-74ef9b552d39/22221f63-b32d-4372-b662-a2ce74004c9b"
+					(reference "#PWR07")
+					(unit 1)
+				)
+			)
 		)
 	)
@@
 				(path "/3c29357a-68d2-4983-bb91-6d3951934863"
 					(reference "R9")
+					(unit 1)
+				)
+			)
+			(project "TTT"
+				(path "/990e0fce-b73a-47af-aaa3-74ef9b552d39/22221f63-b32d-4372-b662-a2ce74004c9b"
+					(reference "R3")
 					(unit 1)
 				)
@@
 				)
 			)
+			(project "TTT"
+				(path "/990e0fce-b73a-47af-aaa3-74ef9b552d39/22221f63-b32d-4372-b662-a2ce74004c9b"
+					(reference "#PWR09")
+					(unit 1)
+				)
+			)
 		)
 	)
@@
 				)
 			)
+			(project "TTT"
+				(path "/990e0fce-b73a-47af-aaa3-74ef9b552d39/22221f63-b32d-4372-b662-a2ce74004c9b"
+					(reference "Rsnsb1")
+					(unit 1)
+				)
+			)
 		)
 	)
@@
 				)
 			)
+			(project "TTT"
+				(path "/990e0fce-b73a-47af-aaa3-74ef9b552d39/22221f63-b32d-4372-b662-a2ce74004c9b"
+					(reference "#PWR015")
+					(unit 1)
+				)
+			)
 		)
 	)
@@
 					(unit 1)
 				)
+			)
+			(project "TTT"
+				(path "/990e0fce-b73a-47af-aaa3-74ef9b552d39/22221f63-b32d-4372-b662-a2ce74004c9b"
+					(reference "J4")
+					(unit 1)
+				)
