File: LTC4162/LTC4162.kicad_pcb (KiCad board)
At the start: 4 copper layers, 44.3 x 47.6 mm, 17 parts, among them J1 Conn_01x02, J2 Conn_01x02, J3 Conn_01x02, Q6 FDMC8327L, Q7 2N7002

Commit message: Add files via upload
Parts:
- moved Q6 2.67 mm to (138.8, 78.3)
- moved C5 0.44 mm to (146.8, 87.8)
Routing:
- net /CELLS0: track 48.4 -> 19.8 mm
- net /Vin LTC4162: track 44.2 -> 35.2 mm
- net Net-(B4-INFET): track 7.03 -> 9.70 mm
- net /BATSENS+: track 55.3 -> 56.6 mm
- net Net-(Q6-D): track 9.92 -> 11.0 mm
- net Net-(B4-RT): track 4.07 -> 3.37 mm
- net /BATFET: track 20.0 -> 20.5 mm
- added copper zone on F.Cu, net /CELLS0

Commit message: Add files via upload
Parts:
- B4: footprint New:QFN50P400X500X80-29N-D -> LTC4162:QFN50P400X500X80-29N-D
Routing:
- net /Vin LTC4162: track 35.2 -> 45.3 mm
- net GND: track 0.50 -> 4.08 mm
Other:
- board size 44.3 x 47.6 mm -> 44.3 x 45.8 mm

Commit message: Add files via upload
Routing:
- net GND: track 4.08 -> 6.70 mm
- net /BOOST: track 10.8 -> 12.6 mm
