File: MAX17302/MAX17302.kicad_sch (KiCad schematic)
At the start: 12 parts, among them J1 Conn_01x02, J2 Conn_01x02, J3 Conn_01x03, Q1 Q_NMOS_DSG, Q2 Q_NMOS_DSG, U1 MAX17302G+T

Commit message: Update PCB layout and add NTC thermistor
- Resolved clearance issues to ensure design safety.
- Adjusted trace widths for better routing.
- Optimized component placements and overall layout.
- Added NTC thermistor for temperature monitoring.
Parts:
- added TH1: 10kΩ, Resistor_SMD:R_0805_2012Metric, symbol Device:Thermistor_NTC
Connections:
- net GND: now also TH1.1
- net at U1.1 (TH): now also TH1.2
Other:
- note added: "- CP (Chân 2): V ≈ 8V (2 x VBATT) | I = ~µA (Bơm điện tích Charge Pump) - CHG / DIS (Chân 14, 12): V ≈ 8V (Áp kích FET) | I = ~100µA (Điều khiển MOSFET) - REG (Chân 7): V = 1.8V | I = (LDO nội bộ)"
- note added: "- CSP / CSN (Chân 5, 6): V = 2.5V - 4.2V (Đo dòng pin) | I = ±1.5µA (Sụt áp đo lường tối đa ±51.2mV) - BATT (Chân 3): V = 2.16V - 4.9V (Đo áp pin & Nguồn nuôi) | I = 18µA (Hibernate) - 24µA (Active) - TH (Chân 1): V = 0V - 1.8V (Đo nhiệt độ NTC) | I = ~µA - PCKP (Chân 11): V = -0.3V - 18V (Nhận diện sạc/tải) | I = 30µA (Dòng dò tìm)"
- note added: "- Tuyến PCKP → MOSFETs → Sense → BATT: V = 2.5V - 4.2V | I = 3.2A (Dòng sạc/xả hệ thống)"
- note added: "1. NHÓM CHÂN CÔNG SUẤT (DÒNG LỚN) (Lưu ý: Dòng sạc/xả đi qua 2 MOSFET ngoài và điện trở Sense, không qua lõi IC)"
- note added: "2. NHÓM CHÂN ĐO LƯỜNG (DÒNG NHỎ)"
- note added: "3. NHÓM CHÂN ĐIỀU KHIỂN (ÁP CAO, DÒNG NHỎ)"
- moved on the sheet: C1, C2, C3, C4, J1, J2, J3, Q1, Q2, R1, R2

Commit message: Rebuild the MAX17302 PCB
also add new 3D of MAX17302
Parts:
- Q1, Q2: footprint Package_DFN_QFN:DFN-4_5x7mm_P5.08mm -> a:FDMC86139P
- U1: footprint 21-0137I_T1433-2_MXM -> Max17302:21-0137I_T1433-2_MXM
Connections:
- no-connect marks 2 -> 1
Changed lines of the file:
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@@
+	)
+	(junction
+		(at 201.93 92.71)
+		(diameter 0)
+		(color 0 0 0 0)
 	)
 	(junction
@@
 		(color 0 0 0 0)
 	)
-	(junction
-		(at 201.93 92.71)
-		(diameter 0)
-		(color 0 0 0 0)
-	)
 	(no_connect
 		(at 167.64 123.19)
-	)
-	(no_connect
-		(at 196.85 105.41)
 	)
 	(wire
@@
 		(property "Value" "Q_NMOS_DSG"
 			(at 147.828 88.9 90)
+			(hide yes)
 			(show_name no)
 			(do_not_autoplace no)
@@
 			)
 		)
-		(property "Footprint" "Package_DFN_QFN:DFN-4_5x7mm_P5.08mm"
+		(property "Footprint" "a:FDMC86139P"
 			(at 160.02 90.17 0)
 			(hide yes)
@@
 			)
 		)
-		(property "Footprint" "Package_DFN_QFN:DFN-4_5x7mm_P5.08mm"
+		(property "Footprint" "a:FDMC86139P"
 			(at 165.1 90.17 0)
 			(hide yes)
@@
 			)
 		)
-		(property "Footprint" "21-0137I_T1433-2_MXM"
+		(property "Footprint" "Max17302:21-0137I_T1433-2_MXM"
 			(at 167.64 115.57 0)
 			(hide yes)

Commit message: Add files via upload
Parts:
- renumbered C3 to C10, C4 to C11, C1 to C8, C2 to C9, J1 to J5, J2 to J6, J3 to J7, Q1 to Q4, Q2 to Q5, R1 to R4, R2 to R5
Changed lines of the file:
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@@
 		)
 		(instances
+			(project "TTT"
+				(path "/990e0fce-b73a-47af-aaa3-74ef9b552d39/44791df6-96ae-4f24-a49d-da257675e590"
+					(reference "#PWR04")
+					(unit 1)
+				)
+			)
 			(project "MAX17302"
 				(path "/db8ca071-62bf-4378-b43c-6ff789ff64b4"
@@
 		(dnp no)
 		(fields_autoplaced yes)
-		(property "Reference" "J3"
+		(property "Reference" "J7"
 			(at 260.35 128.2699 0)
 			(show_name no)
@@
 		)
 		(instances
+			(project "TTT"
+				(path "/990e0fce-b73a-47af-aaa3-74ef9b552d39/44791df6-96ae-4f24-a49d-da257675e590"
+					(reference "J7")
+					(unit 1)
+				)
+			)
 			(project "MAX17302"
 				(path "/db8ca071-62bf-4378-b43c-6ff789ff64b4"
@@
 		(dnp no)
 		(fields_autoplaced yes)
-		(property "Reference" "J2"
+		(property "Reference" "J6"
 			(at 204.47 82.5499 0)
 			(show_name no)
@@
 		)
 		(instances
+			(project "TTT"
+				(path "/990e0fce-b73a-47af-aaa3-74ef9b552d39/44791df6-96ae-4f24-a49d-da257675e590"
+					(reference "J6")
+					(unit 1)
+				)
+			)
 			(project "MAX17302"
 				(path "/db8ca071-62bf-4378-b43c-6ff789ff64b4"
@@
 		(dnp no)
 		(fields_autoplaced yes)
-		(property "Reference" "J1"
+		(property "Reference" "J5"
 			(at 132.08 107.95 0)
 			(show_name no)
@@
 		)
 		(instances
+			(project "TTT"
+				(path "/990e0fce-b73a-47af-aaa3-74ef9b552d39/44791df6-96ae-4f24-a49d-da257675e590"
+					(reference "J5")
+					(unit 1)
+				)
+			)
 			(project "MAX17302"
 				(path "/db8ca071-62bf-4378-b43c-6ff789ff64b4"
@@
 		)
 		(instances
+			(project "TTT"
+				(path "/990e0fce-b73a-47af-aaa3-74ef9b552d39/44791df6-96ae-4f24-a49d-da257675e590"
+					(reference "#PWR01")
+					(unit 1)
+				)
+			)
 			(project "MAX17302"
 				(path "/db8ca071-62bf-4378-b43c-6ff789ff64b4"
@@
 		(in_pos_files yes)
 		(dnp no)
-		(property "Reference" "C2"
+		(property "Reference" "C9"
 			(at 156.464 126.238 90)
 			(show_name no)
@@
 		)
 		(instances
+			(project "TTT"
+				(path "/990e0fce-b73a-47af-aaa3-74ef9b552d39/44791df6-96ae-4f24-a49d-da257675e590"
+					(reference "C9")
+					(unit 1)
+				)
+			)
 			(project "MAX17302"
 				(path "/db8ca071-62bf-4378-b43c-6ff789ff64b4"
@@
 		)
 		(instances
+			(project "TTT"
+				(path "/990e0fce-b73a-47af-aaa3-74ef9b552d39/44791df6-96ae-4f24-a49d-da257675e590"
+					(reference "#PWR03")
+					(unit 1)
+				)
+			)
 			(project "MAX17302"
 				(path "/db8ca071-62bf-4378-b43c-6ff789ff64b4"
@@
 		(in_pos_files yes)
 		(dnp no)
-		(property "Reference" "C3"
+		(property "Reference" "C10"
 			(at 161.036 118.618 90)
 			(show_name no)
@@
 		)
 		(instances
+			(project "TTT"
+				(path "/990e0fce-b73a-47af-aaa3-74ef9b552d39/44791df6-96ae-4f24-a49d-da257675e590"
+					(reference "C10")
+					(unit 1)
+				)
+			)
 			(project "MAX17302"
 				(path "/db8ca071-62bf-4378-b43c-6ff789ff64b4"
@@
 		)
 		(instances
+			(project "TTT"
+				(path "/990e0fce-b73a-47af-aaa3-74ef9b552d39/44791df6-96ae-4f24-a49d-da257675e590"
+					(reference "TH1")
+					(unit 1)
+				)
+			)
 			(project "MAX17302"
 				(path "/db8ca071-62bf-4378-b43c-6ff789ff64b4"
@@
 		(in_pos_files yes)
 		(dnp no)
-		(property "Reference" "R2"
+		(property "Reference" "R5"
 			(at 219.71 86.36 90)
 			(show_name no)
@@
 		)
 		(instances
+			(project "TTT"
+				(path "/990e0fce-b73a-47af-aaa3-74ef9b552d39/44791df6-96ae-4f24-a49d-da257675e590"
+					(reference "R5")
+					(unit 1)
+				)
+			)
 			(project "MAX17302"
 				(path "/db8ca071-62bf-4378-b43c-6ff789ff64b4"
@@
 		)
 		(instances
+			(project "TTT"
+				(path "/990e0fce-b73a-47af-aaa3-74ef9b552d39/44791df6-96ae-4f24-a49d-da257675e590"
+					(reference "#PWR02")
+					(unit 1)
+				)
+			)
 			(project "MAX17302"
 				(path "/db8ca071-62bf-4378-b43c-6ff789ff64b4"
@@
 		(in_pos_files yes)
 		(dnp no)
-		(property "Reference" "C4"
+		(property "Reference" "C11"
 			(at 225.044 123.698 90)
 			(show_name no)
@@
 		)
 		(instances
+			(project "TTT"
+				(path "/990e0fce-b73a-47af-aaa3-74ef9b552d39/44791df6-96ae-4f24-a49d-da257675e590"
+					(reference "C11")
+					(unit 1)
+				)
+			)
 			(project "MAX17302"
 				(path "/db8ca071-62bf-4378-b43c-6ff789ff64b4"
@@
 		(dnp no)
 		(fields_autoplaced yes)
-		(property "Reference" "R1"
+		(property "Reference" "R4"
 			(at 181.61 95.2499 0)
 			(show_name no)
@@
 		)
 		(instances
+			(project "TTT"
+				(path "/990e0fce-b73a-47af-aaa3-74ef9b552d39/44791df6-96ae-4f24-a49d-da257675e590"
+					(reference "R4")
+					(unit 1)
+				)
+			)
 			(project "MAX17302"
 				(path "/db8ca071-62bf-4378-b43c-6ff789ff64b4"
@@
 		(in_pos_files yes)
 		(dnp no)
-		(property "Reference" "C1"
+		(property "Reference" "C8"
 			(at 147.32 112.268 90)
 			(show_name no)
@@
 		)
 		(instances
+			(project "TTT"
+				(path "/990e0fce-b73a-47af-aaa3-74ef9b552d39/44791df6-96ae-4f24-a49d-da257675e590"
+					(reference "C8")
+					(unit 1)
+				)
+			)
 			(project "MAX17302"
 				(path "/db8ca071-62bf-4378-b43c-6ff789ff64b4"
@@
 		(in_pos_files yes)
 		(dnp no)
-		(property "Reference" "Q1"
+		(property "Reference" "Q4"
 			(at 147.828 86.36 90)
 			(show_name no)
@@
 		)
 		(instances
+			(project "TTT"
+				(path "/990e0fce-b73a-47af-aaa3-74ef9b552d39/44791df6-96ae-4f24-a49d-da257675e590"
+					(reference "Q4")
+					(unit 1)
+				)
+			)
 			(project "MAX17302"
 				(path "/db8ca071-62bf-4378-b43c-6ff789ff64b4"
@@
 		(in_pos_files yes)
 		(dnp no)
-		(property "Reference" "Q2"
+		(property "Reference" "Q5"
 			(at 162.814 86.106 90)
 			(show_name no)
@@
 		)
 		(instances
+			(project "TTT"
+				(path "/990e0fce-b73a-47af-aaa3-74ef9b552d39/44791df6-96ae-4f24-a49d-da257675e590"
+					(reference "Q5")
+					(unit 1)
+				)
+			)
 			(project "MAX17302"
 				(path "/db8ca071-62bf-4378-b43c-6ff789ff64b4"
@@
 		)
 		(instances
+			(project "TTT"
+				(path "/990e0fce-b73a-47af-aaa3-74ef9b552d39/44791df6-96ae-4f24-a49d-da257675e590"
+					(reference "U1")
+					(unit 1)
+				)
+			)
 			(project "MAX17302"
 				(path "/db8ca071-62bf-4378-b43c-6ff789ff64b4"
@@
 		)
 	)
-	(sheet_instances
-		(path "/"
-			(page "1")
-		)
-	)
-	(embedded_fonts no)
 )
